Commit message: Initial commit

File: urdf/turtlebot3_burger.urdf (robot description, URDF)
Before this commit: robot turtlebot3_burger, 7 links, 6 joints
Links:
- removed link base_footprint
- removed link base_scan
- removed link caster_back_link
- removed link imu_link
- removed link wheel_left_link
- removed link wheel_right_link
- added link lidar; visual cylinder length=0.1 radius=0.05
- link base_link: mass 8.2573504e-01 -> None; geometry visual box size=0.5 0.5 0.2
Joints:
- removed joint base_joint
- removed joint caster_back_joint
- removed joint imu_joint
- removed joint scan_joint
- removed joint wheel_left_joint
- removed joint wheel_right_joint
- added joint base_to_lidar: type fixed, parent base_link, child lidar, origin xyz=0 0 0.25
